File: NyanCatEarrings.sch (KiCad schematic (older format))
At the start: 11 parts, among them IC1 ATTINY10-TS, P1 GND, P2 VCC, P4 TPI, P5 CLK, P6 RST

Commit message: Update BOM
Parts:
- D1, D2: mfr (none) -> APT1608EC
- IC1: mfr (none) -> ATTINY10-TSHR
- R1: mfr (none) -> ESR03EZPJ101
Changed lines of the file:
@@
 LIBS:contrib
 LIBS:valves
+LIBS:NyanCatEarrings-cache
 EELAYER 25 0
 EELAYER END
@@
 F 2 "LEDs:LED_0603" H 3180 2740 50  0001 C CNN
 F 3 "" H 3180 2740 50  0000 C CNN
+F 4 "APT1608EC" H 3180 2740 60  0001 C CNN "mfr"
 	1    3180 2740
 	1    0    0    -1
@@
 F 2 "Resistors_SMD:R_0603_HandSoldering" V 2735 2740 50  0001 C CNN
 F 3 "" H 2805 2740 50  0000 C CNN
+F 4 "ESR03EZPJ101" V 2805 2740 60  0001 C CNN "mfr"
 	1    2805 2740
 	0    1    1    0
@@
 F 2 "LEDs:LED_0603" H 3190 3015 50  0001 C CNN
 F 3 "" H 3190 3015 50  0000 C CNN
+F 4 "APT1608EC" H 3190 3015 60  0001 C CNN "mfr"
 	1    3190 3015
 	1    0    0    -1
@@
 F 2 "TO_SOT_Packages_SMD:TSOT-23-6_MK06A_HandSoldering" H 5635 3115 50  0000 C CIN
 F 3 "" H 5635 2865 50  0000 C CNN
+F 4 "ATTINY10-TSHR" H 5635 2865 60  0001 C CNN "mfr"
 	1    5635 2865
 	1    0    0    -1

Commit message: Update supercapacitor
Parts:
- BT1: mfr (none) -> MAL219691131E3
Changed lines of the file:
@@
 F 2 "TIH:Supercapcoin" V 7520 2980 50  0001 C CNN
 F 3 "" V 7520 2980 50  0000 C CNN
+F 4 "MAL219691131E3" H 7520 2920 60  0001 C CNN "mfr"
 	1    7520 2920
 	1    0    0    -1
